File: get-a-grip-on-reality/MCU.kicad_sch (KiCad schematic)
At the start: 0 parts

Commit message: add mcu schematic
Parts:
- added C1: 10u, symbol Device:C
- added C2, C3: 1u, symbol Device:C
- added D1: LED, symbol Device:LED
- added R1: 500, symbol Device:R
- added U3: ESP32-S3-WROOM-1, esp32-s3-wroom-1:ESP32-S3-WROOM-1-N8_EXP, symbol Espressif:ESP32-S3-WROOM-1
Connections:
- new net: D1.1 (K), R1.1
- new net: D1.2 (A), U3.16 (GPIO46)
- new net +3.3V: C1.1, C2.1, C3.1, U3.2 (3V3), U3.3 (EN)
- new net GND: C1.2, C2.2, C3.2, R1.2, U3.1 (GND), U3.40 (GND), U3.41 (GND)
- new net IN_1: U3.4 (GPIO4/TOUCH4/ADC1_CH3)
- new net IN_2: U3.5 (GPIO5/TOUCH5/ADC1_CH4)
- new net IN_3: U3.6 (GPIO6/TOUCH6/ADC1_CH5)
- new net IN_4: U3.7 (GPIO7/TOUCH7/ADC1_CH6)
- new net IN_5: U3.8 (GPIO15/U0RTS/ADC2_CH4)
- new net MOTOR_1: U3.32 (MTCK/GPIO39/CLK_OUT3/SUBSPICS1)
- new net MOTOR_2: U3.31 (GPIO38/FSPIWP/SUBSPIWP)
- new net MOTOR_3: U3.30 (SPIDQS/GPIO37/FSPIQ/SUBSPIQ)
- new net MOTOR_4: U3.29 (SPIIO7/GPIO36/FSPICLK/SUBSPICLK)
- new net MOTOR_5: U3.28 (SPIIO6/GPIO35/FSPID/SUBSPID)
- new net USB_P: U3.13 (GPIO19/U1RTS/ADC2_CH8/CLK_OUT2/USB_D-), U3.14 (GPIO20/U1CTS/ADC2_CH9/CLK_OUT1/USB_D+)

Commit message: mcu
Parts:
- added BOOT1, RESET1: SW_Push, symbol Switch:SW_Push
- added C6, C7: 0.1u, symbol Device:C
- added C8, C9: 10u, symbol Device:C
- added D2: LED, symbol Device:LED
- added J2: USB_OTG, symbol Connector:USB_OTG
- added R4: 10k, symbol Device:R
- added R5: 1M, symbol Device:R
- added R6: 200k, symbol Device:R
- added R7: 5.1k, symbol Device:R
- added U4: D3V3XA4B10LP, Package_DFN_QFN:Diodes_UDFN-10_1.0x2.5mm_P0.5mm, symbol Power_Protection:D3V3XA4B10LP
- added U5: TLV75801PDRV, Package_SON:WSON-6-1EP_2x2mm_P0.65mm_EP1x1.6mm, symbol Regulator_Linear:TLV75801PDRV
Connections:
- net +3.3V: now also R4.1; no longer U3.3 (EN)
- net GND: now also BOOT1.1, C6.2, C7.2, C8.2, C9.2, D2.1 (K), R6.2, RESET1.1, U5.3 (GND), U5.7 (GND)
- net at U3.27 (GPIO0/BOOT): now also BOOT1.2, C7.1
- new net: C6.1, R4.2, RESET1.2, U3.3 (EN)
- new net: J2.1 (VBUS), U4.4, U4.7 (NC)
- new net: J2.2 (D-), U4.1, U4.10 (NC)
- new net: J2.3 (D+), U4.2, U4.9 (NC)
- new net: D2.2 (A), R7.1
- new net: C9.1, R5.1, R7.2, U5.1 (OUT)
- new net: R5.2, R6.1, U5.2 (FB)
- new net: C8.1, U5.4 (EN), U5.6 (IN)
- new net: U4.3 (VSS), U4.8 (VSS)
Other:
- note added: "3V3"
- note added: "5VUSB"
- note added: "USB_N"
- note added: "USB_P"
