File: get-a-grip-on-reality/MCU.kicad_sch (KiCad schematic)
At the start: 22 parts, among them J12 Battery Connector MCU, J13 Conn_01x05_Pin, P1 USB_C_Plug_USB2.0, U1 TLV76733DRVx, U2 ESP32-S3-WROOM-1, U3 D3V3XA4B10LP

Commit message: finish pcb no drc errors
Connections:
- net +5V: now also J12.2 (Pin_2); no longer J12.1 (Pin_1)
- net GND: now also J12.1 (Pin_1); no longer J12.2 (Pin_2)
Changed lines of the file:
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@@
 	(symbol
 		(lib_id "Connector:Conn_01x02_Socket")
-		(at 104.14 172.72 0)
+		(at 104.14 175.26 0)
+		(mirror x)
 		(unit 1)
 		(exclude_from_sim no)
@@
 		(on_board yes)
 		(dnp no)
-		(fields_autoplaced yes)
 		(property "Reference" "J12"
-			(at 105.41 173.355 0)
+			(at 105.41 174.625 0)
 			(effects
 				(font
@@
 		)
 		(property "Value" "Battery Connector MCU"
-			(at 105.41 175.895 0)
+			(at 105.41 172.085 0)
 			(effects
 				(font
@@
 		)
 		(property "Footprint" "Connector_AMASS:AMASS_XT30PW-M_1x02_P2.50mm_Horizontal"
-			(at 104.14 172.72 0)
+			(at 104.14 175.26 0)
 			(effects
 				(font
@@
 		)
 		(property "Datasheet" "~"
-			(at 104.14 172.72 0)
+			(at 104.14 175.26 0)
 			(effects
 				(font
@@
 		)
 		(property "Description" ""
-			(at 104.14 172.72 0)
+			(at 104.14 175.26 0)
 			(effects
 				(font

Commit message: fixes to pcb
Connections:
- net +5V: no longer P1.A4 (VBUS), P1.A9 (VBUS), P1.B4 (VBUS), P1.B9 (VBUS), U3.4, U3.7 (NC)
- net GND: now also P1.S1 (SHIELD)
- new net +5V_USB_ESP: P1.A4 (VBUS), P1.A9 (VBUS), P1.B4 (VBUS), P1.B9 (VBUS), U3.4, U3.7 (NC)
- no-connect marks 7 -> 6
Changed lines of the file:
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@@
 	)
 	(junction
+		(at 224.79 120.65)
+		(diameter 0)
+		(color 0 0 0 0)
+	)
+	(junction
 		(at 30.48 166.37)
 		(diameter 0)
@@
 	)
 	(no_connect
-		(at 217.17 120.65)
-	)
-	(no_connect
 		(at 83.82 124.46)
 	)
@@
 	(wire
 		(pts
+			(xy 217.17 120.65) (xy 224.79 120.65)
+		)
+		(stroke
+			(width 0)
+			(type default)
+		)
+	)
+	(wire
+		(pts
 			(xy 77.47 81.28) (xy 83.82 81.28)
 		)
@@
 		(on_board yes)
 		(dnp no)
-		(property "Reference" "#PWR043"
+		(property "Reference" "#PWR5VUSB_ESP0101"
 			(at 279.4 83.82 0)
 			(effects
@@
 			)
 		)
-		(property "Value" "+5V"
+		(property "Value" "+5V_USB_ESP"
 			(at 279.4 74.93 0)
 			(effects
@@
 			(project "get-a-grip-on-reality"
 				(path "/baa0c64e-005f-4609-8fc2-3159870af962/ac4bf6b8-92c6-4d58-8d59-9dba1bb4caf0"
-					(reference "#PWR043")
+					(reference "#PWR5VUSB_ESP0101")
 					(unit 1)
 				)
