File: get-a-grip-on-reality/_autosave-MCU.kicad_sch (KiCad schematic)
At the start: 20 parts, among them J2 USB_OTG, U3 ESP32-S3-WROOM-1, U4 D3V3XA4B10LP, U5 TLV75801PDRV

Commit message: add new chips
Parts:
- removed C9: 10u, symbol Device:C
- removed R5: 1M, symbol Device:R
- removed R6: 200k, symbol Device:R
- removed U5: TLV75801PDRV, Package_SON:WSON-6-1EP_2x2mm_P0.65mm_EP1x1.6mm, symbol Regulator_Linear:TLV75801PDRV
- added C4, C5: 1u, symbol Device:C
- added D4: ESD9B3.3ST5G, Diode_SMD:D_SOD-923, symbol Diode:ESD9B3.3ST5G
- added U1: TLV76733DRVx, Package_SON:WSON-6-1EP_2x2mm_P0.65mm_EP1x1.6mm_ThermalVias, symbol Regulator_Linear:TLV76733DRVx
- C8: value 10u -> 1u
Connections:
- net +3.3V: now also C8.1, C5.1, D4.2 (A2), U1.1 (OUT), U1.2 (SNS)
- net +5V: now also C4.1, U1.4 (EN), U1.6 (IN); no longer C8.1
- net GND: now also U4.3 (VSS), U4.8 (VSS), C4.2, C5.2, D4.1 (A1), U1.3 (GND), U1.5 (GND), U1.7 (PAD)
