File: get-a-grip-on-reality/_autosave-Power.kicad_sch (KiCad schematic)
At the start: 16 parts, among them J1 Battery Connector, J4 Conn_01x05_Pin, U2 BQ25887

Commit message: add new chips
Connections:
- no-connect marks 3 -> 4
Other:
- note removed: "Battery Charging"
