File: get-a-grip-on-reality/get-a-grip-on-reality.kicad_pcb (KiCad board)
At the start: 2 copper layers, 100 x 100 mm, 87 parts, among them J1 Conn_01x04_Pin, J10 MOTOR4, J11 MOTOR5, J12 Battery Connector MCU, J13 Conn_01x05_Pin, J14 Conn_01x05_Pin, J15 Battery Connector Bat, J2 HALL1, J3 HALL2, J4 HALL3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

Commit message: more comments
Routing:
- net GND: vias 704 -> 706
Other:
- board text added: "< Avoid silkscreen on pads"
- board text added: "< Give a bit more width here"
- board text added: "< Just route 5v, no need for polyfill"
- board text added: "< Move this closer to U6"
- board text added: "< Move this via over for better GND path for servos"
- board text added: "< Put this closer to the IC above the resistors Reroute the 5v since its cutting through a lot See the datasheet recommended layout"
- board text added: "< Rotate this so GND has a better path to U7"
- board text added: "< This decouples U4, but its all the way out here"
- board text added: "< We dont need all these vias here"
- board text added: "< move this, then move C12/R6 closer"
- board text added: "<Add vias here or reduce polyfill area Bottom part of poly not doing anything"
- board text added: "Add C9 cap here>"
- board text added: "Gr right angle>"
- board text added: "Make the GND routing better > Dont via the pad"
- board text added: "Make this thicker>"
- board text added: "You can put the 10uF with the 1uF, no need to put it under>"
- board text added: "move the header up instead > Move the cap closer to the IC"

Commit message: implement all of winstons comments
Parts:
- C7: moved to F.Cu
- moved C9 23.6 mm to (54.2, 43.0), turned to -90 degrees
- moved C7 20.0 mm to (42.9, 70.1), turned to 180 degrees
- moved C8 10.6 mm to (46.7, 44.9)
- moved C14 7.59 mm to (125.4, 54.6)
- moved R3 7.01 mm to (74.2, 61.9), turned to -90 degrees
- moved C12 3.85 mm to (74.2, 55.0)
- moved R6 3.85 mm to (74.2, 53.0)
- moved R16 3.69 mm to (108.3, 63.8)
- moved C23 2.95 mm to (100.5, 62.3), turned to -90 degrees
- moved C16 2.94 mm to (117.6, 61.3)
- moved C19 2.93 mm to (115.5, 61.3)
- moved J1 2.85 mm to (46.7, 42.0)
- moved R20 2.59 mm to (104.4, 62.3), turned to -90 degrees
- moved D7 2.22 mm to (128.4, 53.0), turned to 0 degrees
- moved C15 1.72 mm to (119.7, 61.3)
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Routing:
- net GND: track 50.6 -> 36.2 mm, vias 706 -> 226
- net +5V: track 67.9 -> 78.6 mm
- net Net-(U5-1OUT): track 11.5 -> 6.83 mm
- net +3.3V: track 127.8 -> 124.1 mm, vias 1 -> 0
- net /IMU/SDO: track 11.1 -> 14.3 mm
- net Net-(U7-SS): track 7.15 -> 4.04 mm
- net Net-(U6-BTST): track 11.6 -> 13.8 mm
- net Net-(U7-VCC): track 14.9 -> 13.0 mm
- net /MOTOR1: track 12.8 -> 14.7 mm
- net /IMU/SCLK: track 16.7 -> 18.5 mm
- net Net-(U7-PG): track 4.69 -> 6.10 mm
- net Net-(U7-FB): track 6.52 -> 5.18 mm
- net Net-(U7-ILIM): track 2.01 -> 3.32 mm
- net /Light Sensor/1IN-: track 23.4 -> 22.4 mm
- net Net-(U7-MSEL): track 6.29 -> 5.50 mm
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Other:
- board text removed: "< Give a bit more width here"
- board text removed: "< Just route 5v, no need for polyfill"
- board text removed: "< Move this closer to U6"
- board text removed: "< Move this via over for better GND path for servos"
- board text removed: "< Put this closer to the IC above the resistors Reroute the 5v since its cutting through a lot See the datasheet recommended layout"
- board text removed: "< Rotate this so GND has a better path to U7"
- board text removed: "< This decouples U4, but its all the way out here"
- board text removed: "< We dont need all these vias here"
- board text removed: "< move this, then move C12/R6 closer"
- board text removed: "<Add vias here or reduce polyfill area Bottom part of poly not doing anything"
- board text removed: "Add C9 cap here>"
- board text removed: "Gr right angle>"
- board text removed: "Make the GND routing better > Dont via the pad"
- board text removed: "Make this thicker>"
- board text removed: "You can put the 10uF with the 1uF, no need to put it under>"
- board text removed: "move the header up instead > Move the cap closer to the IC"
