File: get-a-grip-on-reality/get-a-grip-on-reality.kicad_sch (KiCad schematic)
At the start: 0 parts

Commit message: add output
Parts:
- added J10, J11, J12, J13, J14: Conn_01x03_Pin, Connector_PinHeader_2.54mm:PinHeader_1x03_P2.54mm_Vertical, symbol Connector:Conn_01x03_Pin
- added J3: Conn_01x04_Pin, symbol Connector:Conn_01x04_Pin
- added J5: HALL1, symbol Connector:Conn_01x05_Pin
- added J6: HALL2, symbol Connector:Conn_01x05_Pin
- added J7: HALL3, symbol Connector:Conn_01x05_Pin
- added J8: HALL4, symbol Connector:Conn_01x05_Pin
- added J9: HALL5, symbol Connector:Conn_01x05_Pin
Connections:
- new net +3.3V: J3.1 (Pin_1), J5.1 (Pin_1), J6.1 (Pin_1), J7.1 (Pin_1), J8.1 (Pin_1), J9.1 (Pin_1)
- new net +5V: J10.3 (Pin_3), J11.3 (Pin_3), J12.3 (Pin_3), J13.3 (Pin_3), J14.3 (Pin_3)
- new net GND: J10.1 (Pin_1), J11.1 (Pin_1), J12.1 (Pin_1), J13.1 (Pin_1), J14.1 (Pin_1), J3.4 (Pin_4), J5.5 (Pin_5), J6.5 (Pin_5), J7.5 (Pin_5), J8.5 (Pin_5), J9.5 (Pin_5)
- new net HALL1A: J5.2 (Pin_2)
- new net HALL1B: J5.3 (Pin_3)
- new net HALL1C: J5.4 (Pin_4)
- new net HALL2A: J6.2 (Pin_2)
- new net HALL2B: J6.3 (Pin_3)
- new net HALL2C: J6.4 (Pin_4)
- new net HALL3A: J7.2 (Pin_2)
- new net HALL3B: J7.3 (Pin_3)
- new net HALL3C: J7.4 (Pin_4)
- new net HALL4A: J8.2 (Pin_2)
- new net HALL4B: J8.3 (Pin_3)
- new net HALL4C: J8.4 (Pin_4)
- new net HALL5A: J9.2 (Pin_2)
- new net HALL5B: J9.3 (Pin_3)
- new net HALL5C: J9.4 (Pin_4)
- new net IMU/SCLK: J3.3 (Pin_3)
- new net IMU/SDO: J3.2 (Pin_2)
- new net MOTOR1: J10.2 (Pin_2)
- new net MOTOR2: J11.2 (Pin_2)
- new net MOTOR3: J12.2 (Pin_2)
- new net MOTOR4: J13.2 (Pin_2)
- new net MOTOR5: J14.2 (Pin_2)
Other:
- sheet Inputs renamed IMU
- removed sheet Drivers
- removed sheet Motors
- added sheet Light Sensor (light.kicad_sch)
- sheet IMU: file Inputs.kicad_sch -> imu.kicad_sch
- sheet IMU ports: added INT1, INT2, SCLK, SCS, SDI, SDO; removed none
- sheet MCU ports: added HALL, INT1, INT2, MOTOR, SCLK, SCS, SDI, SDO; removed none

Commit message: add more to pcb
Parts:
- J1: renamed from J5; footprint (none) -> Connector_JST:JST_SH_BM05B-SRSS-TB_1x05-1MP_P1.00mm_Vertical
- J10: renamed from J13; value Conn_01x03_Pin -> MOTOR4
- J11: renamed from J14; value Conn_01x03_Pin -> MOTOR5
- J2: renamed from J6; footprint (none) -> Connector_JST:JST_SH_BM05B-SRSS-TB_1x05-1MP_P1.00mm_Vertical
- J3: renamed from J7; footprint (none) -> Connector_JST:JST_SH_BM05B-SRSS-TB_1x05-1MP_P1.00mm_Vertical
- J4: renamed from J8; footprint (none) -> Connector_JST:JST_SH_BM05B-SRSS-TB_1x05-1MP_P1.00mm_Vertical
- J5: renamed from J9; footprint (none) -> Connector_JST:JST_SH_BM05B-SRSS-TB_1x05-1MP_P1.00mm_Vertical
- J6: renamed from J3; footprint (none) -> Connector_PinHeader_2.54mm:PinHeader_1x04_P2.54mm_Vertical
- J7: renamed from J10; value Conn_01x03_Pin -> MOTOR1
- J8: renamed from J11; value Conn_01x03_Pin -> MOTOR2
- J9: renamed from J12; value Conn_01x03_Pin -> MOTOR3
Connections:
- net +3.3V: now also J1.5 (Pin_5), J2.5 (Pin_5), J3.5 (Pin_5), J4.5 (Pin_5), J5.5 (Pin_5); no longer J1.1 (Pin_1), J2.1 (Pin_1), J3.1 (Pin_1), J4.1 (Pin_1), J5.1 (Pin_1)
- net +5V: now also J10.1 (Pin_1), J11.1 (Pin_1), J7.1 (Pin_1), J8.1 (Pin_1), J9.1 (Pin_1); no longer J10.3 (Pin_3), J11.3 (Pin_3), J7.3 (Pin_3), J8.3 (Pin_3), J9.3 (Pin_3)
- net GND: now also J1.1 (Pin_1), J10.3 (Pin_3), J11.3 (Pin_3), J2.1 (Pin_1), J3.1 (Pin_1), J4.1 (Pin_1), J5.1 (Pin_1), J7.3 (Pin_3), J8.3 (Pin_3), J9.3 (Pin_3); no longer J1.5 (Pin_5), J10.1 (Pin_1), J11.1 (Pin_1), J2.5 (Pin_5), J3.5 (Pin_5), J4.5 (Pin_5), J5.5 (Pin_5), J7.1 (Pin_1), J8.1 (Pin_1), J9.1 (Pin_1)
- net HALL1A: now also J1.4 (Pin_4); no longer J1.2 (Pin_2)
- net HALL1C: now also J1.2 (Pin_2); no longer J1.4 (Pin_4)
- net HALL2A: now also J2.4 (Pin_4); no longer J2.2 (Pin_2)
- net HALL2C: now also J2.2 (Pin_2); no longer J2.4 (Pin_4)
- net HALL3A: now also J3.4 (Pin_4); no longer J3.2 (Pin_2)
- net HALL3C: now also J3.2 (Pin_2); no longer J3.4 (Pin_4)
- net HALL4A: now also J4.4 (Pin_4); no longer J4.2 (Pin_2)
- net HALL4C: now also J4.2 (Pin_2); no longer J4.4 (Pin_4)
- net HALL5A: now also J5.4 (Pin_4); no longer J5.2 (Pin_2)
- net HALL5C: now also J5.2 (Pin_2); no longer J5.4 (Pin_4)
Other:
- sheet MCU ports: added HALL1A, HALL1B, HALL1C, HALL2A, HALL2B, HALL2C, HALL3A, HALL3B, HALL3C, HALL4A, HALL4B, HALL4C, HALL5A, HALL5B, HALL5C, MOTOR1, MOTOR2, MOTOR3, MOTOR4, MOTOR5; removed HALL, MOTOR
- moved on the sheet: J1, J10, J11, J2, J3, J4, J5, J7, J8, J9

Commit message: fix schematic with winstons suggestions
Parts:
- renumbered J6 to J1, J1 to J2, J2 to J3, J3 to J4, J4 to J5, J5 to J6

Commit message: finish top pcb
Other:
- sheet Light Sensor ports: added LIGHT_OUT; removed none
- sheet MCU ports: added LIGHT_IN; removed none
- note added: "Get a Grip on Reality"
Changed lines of the file:
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@@
+	(wire
+		(pts
+			(xy 156.21 113.03) (xy 179.07 113.03)
+		)
+		(stroke
+			(width 0)
+			(type default)
+		)
+	)
 	(wire
 		(pts
@@
 			(width 0)
 			(type default)
+		)
+	)
+	(text "Get a Grip on Reality"
+		(exclude_from_sim no)
+		(at 220.218 174.244 0)
+		(effects
+			(font
+				(size 5.08 5.08)
+				(thickness 0.7112)
+				(bold yes)
+			)
 		)
 	)
@@
 			)
 		)
+		(pin "LIGHT_OUT" output
+			(at 179.07 113.03 180)
+			(effects
+				(font
+					(size 1.27 1.27)
+				)
+				(justify left)
+			)
+		)
 		(instances
 			(project "get-a-grip-on-reality"
@@
 			)
 		)
+		(pin "LIGHT_IN" input
+			(at 156.21 113.03 0)
+			(effects
+				(font
+					(size 1.27 1.27)
+				)
+				(justify right)
+			)
+		)
