File: get-a-grip-on-reality/imu.kicad_sch (KiCad schematic)
At the start: 4 parts, among them U6 IIM-42652

Commit message: add more to pcb
Parts:
- C10: renamed from C27; footprint (none) -> Capacitor_SMD:C_0805_2012Metric
- C11: renamed from C28; footprint (none) -> Capacitor_SMD:C_0805_2012Metric
- C9: renamed from C26; footprint (none) -> Capacitor_SMD:C_0805_2012Metric
- renumbered U6 to U4
Changed lines of the file:
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@@
 		(dnp no)
 		(fields_autoplaced yes)
-		(property "Reference" "#PWR040"
+		(property "Reference" "#PWR044"
 			(at 180.34 104.14 0)
 			(effects
@@
 			(project "get-a-grip-on-reality"
 				(path "/baa0c64e-005f-4609-8fc2-3159870af962/9a9bf700-d10a-497d-8bed-32e73fee329a"
-					(reference "#PWR040")
+					(reference "#PWR044")
 					(unit 1)
 				)
@@
 		(dnp no)
 		(fields_autoplaced yes)
-		(property "Reference" "C27"
+		(property "Reference" "C10"
 			(at 195.58 107.9499 0)
 			(effects
@@
 			)
 		)
-		(property "Footprint" ""
+		(property "Footprint" "Capacitor_SMD:C_0805_2012Metric"
 			(at 192.7352 113.03 0)
 			(effects
@@
 			(project "get-a-grip-on-reality"
 				(path "/baa0c64e-005f-4609-8fc2-3159870af962/9a9bf700-d10a-497d-8bed-32e73fee329a"
-					(reference "C27")
+					(reference "C10")
 					(unit 1)
 				)
@@
 		(dnp no)
 		(fields_autoplaced yes)
-		(property "Reference" "C26"
+		(property "Reference" "C9"
 			(at 184.15 107.9499 0)
 			(effects
@@
 			)
 		)
-		(property "Footprint" ""
+		(property "Footprint" "Capacitor_SMD:C_0805_2012Metric"
 			(at 181.3052 113.03 0)
 			(effects
@@
 			(project ""
 				(path "/baa0c64e-005f-4609-8fc2-3159870af962/9a9bf700-d10a-497d-8bed-32e73fee329a"
-					(reference "C26")
+					(reference "C9")
 					(unit 1)
 				)
@@
 		(dnp no)
 		(fields_autoplaced yes)
-		(property "Reference" "#PWR039"
+		(property "Reference" "#PWR042"
 			(at 140.97 92.71 0)
 			(effects
@@
 			(project ""
 				(path "/baa0c64e-005f-4609-8fc2-3159870af962/9a9bf700-d10a-497d-8bed-32e73fee329a"
-					(reference "#PWR039")
+					(reference "#PWR042")
 					(unit 1)
 				)
@@
 		(dnp no)
 		(fields_autoplaced yes)
-		(property "Reference" "U6"
+		(property "Reference" "U4"
 			(at 143.1641 120.65 0)
 			(effects
@@
 			(project ""
 				(path "/baa0c64e-005f-4609-8fc2-3159870af962/9a9bf700-d10a-497d-8bed-32e73fee329a"
-					(reference "U6")
+					(reference "U4")
 					(unit 1)
 				)
@@
 		(dnp no)
 		(fields_autoplaced yes)
-		(property "Reference" "#PWR038"
+		(property "Reference" "#PWR043"
 			(at 140.97 133.35 0)
 			(effects
@@
 			(project ""
 				(path "/baa0c64e-005f-4609-8fc2-3159870af962/9a9bf700-d10a-497d-8bed-32e73fee329a"
-					(reference "#PWR038")
+					(reference "#PWR043")
 					(unit 1)
 				)
@@
 		(dnp no)
 		(fields_autoplaced yes)
-		(property "Reference" "C28"
+		(property "Reference" "C11"
 			(at 207.01 107.9499 0)
 			(effects
@@
 			)
 		)
-		(property "Footprint" ""
+		(property "Footprint" "Capacitor_SMD:C_0805_2012Metric"
 			(at 204.1652 113.03 0)
 			(effects
@@
 			(project "get-a-grip-on-reality"
 				(path "/baa0c64e-005f-4609-8fc2-3159870af962/9a9bf700-d10a-497d-8bed-32e73fee329a"
-					(reference "C28")
+					(reference "C11")
 					(unit 1)
 				)
@@
 		(dnp no)
 		(fields_autoplaced yes)
-		(property "Reference" "#PWR041"
+		(property "Reference" "#PWR045"
 			(at 180.34 124.46 0)
 			(effects
@@
 			(project "get-a-grip-on-reality"
 				(path "/baa0c64e-005f-4609-8fc2-3159870af962/9a9bf700-d10a-497d-8bed-32e73fee329a"
-					(reference "#PWR041")
-					(unit 1)
-				)
+					(reference "#PWR045")
+					(unit 1)
+				)
