File: get-a-grip-on-reality/light.kicad_sch (KiCad schematic)
At the start: 0 parts

Commit message: finish top pcb
Parts:
- added C12: 5p, Capacitor_SMD:C_0805_2012Metric, symbol Device:C
- added C13: 10n, Capacitor_SMD:C_0805_2012Metric, symbol Device:C
- added D4, D5, D6: BPV22NF, BPV22NF:XDCR_BPV22NF, symbol BPV22NF:BPV22NF
- added R4: 3k, Resistor_SMD:R_0805_2012Metric, symbol Device:R
- added R5, R7: 47k, Resistor_SMD:R_0805_2012Metric, symbol Device:R
- added R6: 100k, Resistor_SMD:R_0805_2012Metric, symbol Device:R
- added U5: TLV2462CDR, fydp:SOIC127P599X175-8N, symbol TLV2462CDR:TLV2462CDR
Connections:
- new net: C12.2, C13.1, R6.2, U5.1 (1OUT)
- new net +3.3V: U5.8 (VDD+)
- new net 1IN-: C12.1, D4.K, D5.K, D6.K, R6.1, U5.2 (1IN-)
- new net 2IN+: C13.2, R7.2, U5.5 (2IN+)
- new net 2IN-: R4.2, R5.2, U5.6 (2IN-)
- new net GND: D4.A, D5.A, D6.A, R4.1, R7.1, U5.3 (1IN+), U5.4 (GND)
- new net LIGHT_OUT: R5.1, U5.7 (2OUT)
